File: PinguinoHDK.brd (EAGLE design)
At the start: 180.3 x 158.8 mm, 31 parts, among them IC1 7806T, IC2 7805T, IC3 7803T

Commit message: Algunas actualizaciones al cableado de la lcd 16x2
Parts:
- removed C10, C12, C13, C5, C6, C7, C9: 100nf, rcl:C050-024X044
- removed C11, C14, C8: 100uf, rcl:E2,5-5
- removed F1: 2amp, special:FUSE
- removed J1: (no value), con-jack:DCJ0303
- removed L1, L2, L3, L4: 100uH, rcl:0207/10
- removed LED2, LED3: (no value), adafruit:LED3MM
- added BAT1: (no value), SparkFun:BATTCOM_20MM_PTH
- added D1: 1N4007, adafruit:DO41-10
- added D2, D3, D4, D5: 1N4007, diode:DO35-7
- added D6: 4007, diode:DO35-7
- added DZ1: LB10, led:LB10
- added I2C, UART: (no value), SparkFun:1X04_LONGPADS
- added IC4: 74LS155N, 74xx-us:DIL16
- added IC5: 7805, v-reg:78XXL
- added JP1: Sensores Externos, SparkFun:1X06_LONGPADS
- added JP2: (no value), SparkFun:1X02_LONGPADS
- added K1: CQ1-12V, relay:CQ1
- added LM35: LM35CZ, lm35:TO92
- added POT1, POT2, POT3, POT5: 5k, SparkFun:TRIM_POT_PTH
- added Q1: (no value), crystal:TC38H
- added Q2: 2N2222, SparkFun:TO-92
- added R10, R11, R12, R13, R14, R15, R16, R17, R18, R8: 470, SparkFun:AXIAL-0.3-KIT
- added R19: PHOTOCELLPTH, SparkFun:PHOTOCELL
- added R20: 10k, rcl:0204/5@1
- added R21, R22, R24, R28, R7, R9: 4.7k, SparkFun:AXIAL-0.3-KIT
- added R29: 1k, SparkFun:AXIAL-0.3-KIT
- added R5, R6: 1k, rcl:0204/7
- added RESET: (no value), switch-omron:B3F-10XX
- added SERVOS, SERVOS1: (no value), SparkFun:1X03_LONGPADS
- added SG1: BUZZERPTH, SparkFun:BUZZER-12MM
- added T1, T2: 2N3904, transistor:TO92
- added T3: 2SC1815, transistor:TO92-ECB
- added U$1: (no value), keypad4x4_ece:KEYPAD4X4
- added U$2: XBEE, adafruit:XBEE
- added U$4: DS1307, aasanchez:PDIP8
- added U1: LCD-16X2SILK, SparkFun:LCD-16X2
- added X1: (no value), con-wago-508:W237-3E
- added X2, X3: (no value), con-wago-508:W237-132
- added XB1: XBEE-PRO, maxstream:XBEE-PRO
- C1: value 100nf -> 0.1uf; device rcl:C050-024X044 -> SparkFun:CAP-PTH-SMALL2
- C2: value 470uf -> 220nf; device rcl:E2,5-7 -> SparkFun:CPOL-RADIAL-10UF-25V
- C3: value 100nf -> 0.33uf/50v; device rcl:C050-024X044 -> SparkFun:CPOL-RADIAL-10UF-25V
- C4: value 100uf -> 0.1uf; device rcl:E2,5-5 -> SparkFun:CAP-PTH-SMALL2
- IC1: value 7806T -> L293B; device adafruit:TO220H -> st-microelectronics:DIL16
- IC2: value 7805T -> 24AA64P; device adafruit:TO220H -> microchip:DIL8
- IC3: value 7803T -> lm317; device adafruit:TO220H -> v-reg:317TL
- PINGUINOBASE: value PINGUINOBASENO-BORDER -> PINGUINOBASEFACEDOWN; device PinguinoBase:PINGUINOBASE-MIN -> PinguinoBase:FACEDOWN
- R1: value 4.7Ohm/2w -> 1k; device rcl:0414/15 -> SparkFun:AXIAL-0.3-KIT
- R2: value (none) -> 4.7k
- R3: value (none) -> 360
- R4: value (none) -> 240
- moved C1 329.8 mm to (85.1, -174.0), turned to 0 degrees
- moved R1 302.8 mm to (68.6, -180.3), turned to 0 degrees
- moved C2 302.8 mm to (90.2, -163.8), turned to 0 degrees
- moved C4 300.6 mm to (91.4, -174.0)
- moved R4 299.6 mm to (106.7, -180.3)
- moved IC1 297.3 mm to (52.1, -154.9)
- moved LED1 294.7 mm to (29.2, -180.3)
- moved R2 292.4 mm to (81.3, -180.3)
- moved IC3 288.5 mm to (35.6, -142.2)
- moved C3 283.7 mm to (82.5, -163.8)
- moved R3 283.3 mm to (94.0, -180.3)
- moved IC2 219.7 mm to (61.0, -135.9)
- moved PINGUINOBASE 86.4 mm to (106.7, 40.6), flipped to the top, turned to 0 degrees
Connections:
- removed net 12V: C5.1, IC1.1, R1.1
- removed net 12V1: C7.1, C8.+, IC1.3, IC2.1, L2.2
- removed net 3V3: C12.1, L4.1, LED3.A
- removed net 6V: C6.1, L2.1, LED1.A
- removed net N$26: PINGUINOBASE.12
- removed net N$4: C13.1, C14.+, IC3.3, L4.2
- removed net N$43: PINGUINOBASE.11
- removed net N$44: PINGUINOBASE.10
- removed net N$49: PINGUINOBASE.19
- removed net N$50: PINGUINOBASE.18
- removed net N$51: PINGUINOBASE.17
- removed net N$52: PINGUINOBASE.16
- removed net N$53: PINGUINOBASE.15
- removed net N$54: PINGUINOBASE.14
- removed net N$55: PINGUINOBASE.13
- removed net N$57: C1.1, C2.+, F1.2, L1.1
- removed net N$8: LED1.K, R2.P$2
- new net !10: IC1.7, Q2.1, R6.1
- new net +12V: C2.1, C3.1, D2.C, D5.C, D6.C, IC1.8, IC5.IN
- new net +3V3: IC3.2, JP1.1, R4.P$1, XB1.1
- new net +5V: C1.1, C4.1, IC1.16, IC2.8, IC3.3, IC5.OUT, JP1.3, LM35.1, POT1.1, POT2.1, POT3.1, R19.2, R2.P$2, R22.P$1, R29.P$2, R6.2, R7.P$2, R9.P$1, SG1.+, U$4.8
- new net 0: IC2.6, PINGUINOBASE.0, R2.P$1, U$4.6
- new net 1: IC2.5, PINGUINOBASE.1, R7.P$1, U$4.5
- new net 10: IC1.2, R5.2
- new net 11: DZ1.1, IC1.1
- new net 12: DZ1.2, JP2.1
- new net 13: R19.1, R20.2
- new net 14: R1.P$2
- new net 15: JP1.6
- new net 16: JP1.5
- new net 17: JP1.4
- new net 18: POT1.2
- new net 19: POT2.2
- new net 2: IC4.3, PINGUINOBASE.2, R24.P$1
- new net 20: POT3.2
- new net 21: DZ1.3
- new net 22: DZ1.4, PINGUINOBASE.22, U1.4
- new net 23: DZ1.5, PINGUINOBASE.23, U1.15
- new net 24: DZ1.6, PINGUINOBASE.24, U1.14
- new net 25: DZ1.7, PINGUINOBASE.25, U1.13
- new net 26: DZ1.8, PINGUINOBASE.26, U1.12
- new net 27: DZ1.9, PINGUINOBASE.27, U1.11
- new net 28: DZ1.10, PINGUINOBASE.28, U1.6
- new net 3: IC4.13, PINGUINOBASE.3
- new net 4: PINGUINOBASE.4, U$1.5
- new net 5: PINGUINOBASE.5, U$1.6
- new net 6: PINGUINOBASE.6, U$1.7
- new net 7: PINGUINOBASE.7, U$1.8
- new net 8: UART.1
- new net 9: UART.2
- new net N$10: K1.NC, X1.3
- new net N$11: K1.NO, X1.1
- new net N$12: R24.P$2, T1.2
- new net N$14: R28.P$2, T2.2
- new net N$15: D1.A, K1.1, T1.1
- new net N$16: R29.P$1, SG1.-, T2.1
- new net N$18: JP2.2, R28.P$1
- new net N$21: D3.A, IC1.3
- new net N$22: D4.A, IC1.6
- new net N$23: D4.C, D5.A, X2.2
- new net N$24: D2.A, D3.C, X2.1
- new net N$25: D6.A, X3.1
- new net N$27: DZ1.18, R11.P$1
- new net N$28: DZ1.16, R13.P$1
- new net N$29: DZ1.20, R8.P$1
- new net N$30: DZ1.19, R10.P$1
- new net N$31: DZ1.17, R12.P$1
- new net N$32: DZ1.15, R14.P$1
- new net N$33: DZ1.14, R15.P$1
- new net N$34: DZ1.13, R16.P$1
- new net N$35: DZ1.12, R17.P$1
- new net N$36: DZ1.11, R18.P$1
- new net N$37: LED1.A, R22.P$2
- new net N$38: R21.P$1, R9.P$2, U$4.7
- new net N$39: Q2.2, R5.1
- new net N$40: R21.P$2, T3.B
- new net N$41: LED1.K, T3.C
- new net N$42: D1.C, K1.2
- new net RST: RESET.1, RESET.2
- new net VCC: IC4.16
- net 5V: now also PINGUINOBASE.VDD, POT5.1, U1.2; no longer C9.1, L3.1, LED2.A
- net GND: now also BAT1.2, C2.2, C4.2, IC1.10, IC1.12, IC1.13, IC1.15, IC1.4, IC1.5, IC1.9, IC2.1, IC2.3, IC2.4, IC2.7, IC4.8, IC5.GND, JP1.2, LM35.3, PINGUINOBASE.VSS, POT1.3, POT2.3, POT3.3, POT5.3, Q2.3, R10.P$2, R11.P$2, R12.P$2, R13.P$2, R14.P$2, R15.P$2, R16.P$2, R17.P$2, R18.P$2, R20.1, R8.P$2, RESET.3, RESET.4, T2.3, T3.E, U$4.4, U1.1, U1.10, U1.16, U1.5, U1.7, U1.8, U1.9, X3.2, XB1.10; no longer C10.2, C11.-, C12.2, C13.2, C14.-, C2.-, C4.-, C5.2, C6.2, C7.2, C8.-, C9.2, IC1.2, IC3.2, J1.2, J1.3, R2.P$1, R4.P$1
- net N$1: now also LM35.2, R1.P$1; no longer F1.1, J1.1
- net N$2: now also Q1.2, U$4.1; no longer C3.1, C4.+, L1.2, R1.2
- net N$3: now also Q1.1, U$4.2; no longer C10.1, C11.+, IC2.3, IC3.1, L3.2
- net N$45: now also IC4.4, U$1.4; no longer PINGUINOBASE.RST
- net N$46: now also IC4.5, U$1.3; no longer PINGUINOBASE.VSS
- net N$47: now also IC4.6, U$1.2; no longer PINGUINOBASE.VDD
- net N$48: now also IC4.7, U$1.1; no longer PINGUINOBASE.20
- net N$5: now also BAT1.1, U$4.3; no longer LED2.K, R3.P$2
- net N$6: now also POT5.2, U1.3; no longer PINGUINOBASE.22
- net N$7: now also IC3.1, R3.P$2, R4.P$2; no longer PINGUINOBASE.21
- net N$9: now also K1.C, X1.2; no longer LED3.K, R4.P$2
Routing:
- net 5V: track 0.00 -> 311.6 mm
- net GND: track 70.3 -> 296.0 mm
- net 2: track 0.00 -> 206.4 mm
- net 3: track 0.00 -> 194.4 mm
- net 28: track 0.00 -> 192.4 mm
- net 7: track 0.00 -> 190.8 mm
- net 6: track 0.00 -> 180.6 mm
- net 5: track 0.00 -> 178.1 mm
- net 27: track 0.00 -> 177.2 mm
- net 4: track 0.00 -> 175.6 mm
- net 26: track 0.00 -> 172.1 mm
- net 25: track 0.00 -> 167.0 mm
- net 24: track 0.00 -> 156.9 mm
- net 23: track 0.00 -> 151.8 mm
- net 22: track 0.00 -> 129.7 mm
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Other:
- board size 180.3 x 158.8 mm -> 177.8 x 141 mm
