File: PinguinoHDK.sch (EAGLE design)
At the start: 70 parts, among them IC1 L293B, IC2 24AA64P, IC3 lm317, IC5 7805, K1 CQ1-12V, Q2 2N2222, T1 2N3904, T2 2N3904, T3 2SC1815

Commit message: Comienzo de Fuente de Alimentación
Se comenzo a trabajar en la fuente de alimentación, esta esta diseñada
bajo estrictos filtros, para maximizar su eficiencia, el esquematico ya
esta diseñado solo falta la colocacion de los componentes en la placa
Parts:
- removed 4017: 4017N, 40xx:4017N
- removed BAT1: (no value), SparkFun:BATTERY20PTH
- removed D1: 1N4007, adafruit:1N4004
- removed D2, D3, D4, D5: 1N4007, diode:1N4148DO35-7
- removed D6: 4007, diode:1N4148DO35-7
- removed DIS1: TUXGR_16X2_R2, display-lcd:TUXGR_16X2_R2
- removed DZ1: LB10, led:LB10
- removed I2C, UART: (no value), SparkFun:M04LONGPADS
- removed IC5: 7805, v-reg:78XXL
- removed JP1: Sensores Externos, SparkFun:M06LONGPADS
- removed JP2: (no value), SparkFun:M02PTH3
- removed K1: CQ1-12V, relay:CQ1-12V
- removed LM35: LM35CZ, lm35:LM35CZ
- removed PINGUINO: PINGUINOBASENO-BORDER, PinguinoBase:PINGUINOBASENO-BORDER
- removed POT1, POT2, POT3, POT4: 5k, SparkFun:TRIMPOTPTH
- removed Q1: (no value), crystal:CRYSTALTC38H
- removed Q2: 2N2222, SparkFun:TRANSISTOR_NPNTO92
- removed R10, R11, R12, R13, R14, R15, R16, R17, R18, R8: 470, SparkFun:RESISTORKIT
- removed R19: PHOTOCELLPTH, SparkFun:PHOTOCELLPTH
- removed R20: 10k, rcl:R-US_0204/5
- removed R21, R22, R24, R28, R7, R9: 4.7k, SparkFun:RESISTORKIT
- removed R29: 1k, SparkFun:RESISTORKIT
- removed R5, R6: 1k, rcl:R-EU_0204/7
- removed RESET: (no value), switch-omron:10-XX
- removed SERVOS, SERVOS1: (no value), SparkFun:M03LONGPADS
- removed SG1: BUZZERPTH, SparkFun:BUZZERPTH
- removed T1, T2: 2N3904, transistor:2N3904
- removed T3: 2SC1815, transistor:2SC1815
- removed U$1: (no value), keypad4x4_ece:KEYPAD4X4
- removed U$2: DS1307, aasanchez:DS1307
- removed X1: (no value), con-wago-508:W237-3E
- removed X2, X3: (no value), con-wago-508:W237-02P
- removed XB1: XBEE-PRO, maxstream:XBEE-PRO
- added C10, C12, C13, C5, C6, C7, C9: 100nf, rcl:C-EU050-024X044
- added C11, C14, C8: 100uf, rcl:CPOL-USE2.5-5
- added F1: 2amp, special:FUSE
- added J1: (no value), con-jack:DCJ0303
- added L1, L2, L3, L4: 100uH, rcl:L-EU0207/10
- added LED2, LED3: (no value), adafruit:LED3MM
- added PINGUINOBASE: PINGUINOBASENO-BORDER, PinguinoBase:PINGUINOBASENO-BORDER
- C1: value 0.1uf -> 100nf; device SparkFun:CAPPTH2 -> rcl:C-EU050-024X044
- C2: value 220nf -> 470uf; device SparkFun:CAP_POLPTH2 -> rcl:CPOL-USE2.5-7
- C3: value 0.33uf/50v -> 100nf; device SparkFun:CAP_POLPTH2 -> rcl:C-EU050-024X044
- C4: value 0.1uf -> 100uf; device SparkFun:CAPPTH2 -> rcl:CPOL-USE2.5-5
- IC1: value L293B -> 7806T; device st-microelectronics:L293D -> adafruit:7806T
- IC2: value 24AA64P -> 7805T; device microchip:24AA64P -> adafruit:7806T
- IC3: value lm317 -> 7803T; device v-reg:LM317TL -> adafruit:7806T
- R1: value 1k -> 4.7Ohm/2w; device SparkFun:RESISTORKIT -> rcl:R-US_0414/15
- R2: value 4.7k -> (none)
- R3: value 360 -> (none)
- R4: value 240 -> (none)
Connections:
- removed net !10: IC1.2A, Q2.E, R6.1
- removed net +12V: C2.+, C3.+, D2.C, D5.C, D6.C, IC1.VCC2, IC5.IN
- removed net +3V3: IC3.OUT, JP1.1, R4.1, XB1.VCC
- removed net +5V: 4017P.VDD, C1.1, C4.1, DIS1.VCC, IC1.VCC1, IC2.VCC, IC3.IN, IC5.OUT, JP1.3, LM35.+VS, PINGUINO.+5V, POT1.CCW, POT2.CCW, POT3.CCW, POT4.CCW, R19.P$2, R2.2, R22.1, R29.2, R6.2, R7.2, R9.1, SG1.1, U$2.VCC
- removed net 0: IC2.SCL, PINGUINO.SDA-PIN0, R2.1, U$2.SCL
- removed net 1: IC2.SDA, PINGUINO.SCL-PIN1, R7.1, U$2.SDA
- removed net 10: IC1.1A, PINGUINO.PIN10, R5.2
- removed net 11: DZ1-1.A, IC1.1-2EN, PINGUINO.PIN11-PWM
- removed net 12: DZ1-2.A, JP2.1, PINGUINO.PIN12-PWM
- removed net 13: PINGUINO.PIN13/ANALOG-0, R19.P$1, R20.2
- removed net 14: PINGUINO.PIN14/ANALOG-1, R1.2
- removed net 15: JP1.6, PINGUINO.PIN15/ANALOG-2
- removed net 16: JP1.5, PINGUINO.PIN16/ANALOG-3
- removed net 17: JP1.4, PINGUINO.PIN17/ANALOG-4
- removed net 18: PINGUINO.PIN18/ANALOG-5, POT1.WIPER
- removed net 19: PINGUINO.PIN19/ANALOG-6, POT2.WIPER
- removed net 2: PINGUINO.PIN2, R24.1
- removed net 20: PINGUINO.PIN20/ANALOG-7, POT3.WIPER
- removed net 21: DZ1-3.A, PINGUINO.PIN21
- removed net 22: DIS1.RS, DZ1-4.A, PINGUINO.PIN22
- removed net 23: DIS1.E, DZ1-5.A
- removed net 24: DIS1.D4, DZ1-6.A
- removed net 25: DIS1.D5, DZ1-7.A
- removed net 26: DIS1.D6, DZ1-8.A
- removed net 27: DIS1.D7, DZ1-9.A
- removed net 28: DIS1.NC@1, DZ1-10.A
- removed net 3: 4017A.CLK, PINGUINO.PIN3
- removed net 4: PINGUINO.PIN4, U$1.R4
- removed net 5: PINGUINO.PIN5, U$1.R3
- removed net 6: PINGUINO.PIN6, U$1.R2
- removed net 7: PINGUINO.PIN7, U$1.R1
- removed net 8: UART.1
- removed net 9: UART.2
- removed net N$10: K12.O, X1-3.KL
- removed net N$11: K12.S, X1-1.KL
- removed net N$12: R24.2, T1.B
- removed net N$13: 4017A.Q2, U$1.C2
- removed net N$14: R28.2, T2.B
- removed net N$15: D1.A, K11.1, T1.C
- removed net N$16: R29.1, SG1.2, T2.C
- removed net N$17: 4017A.Q3, U$1.C1
- removed net N$18: JP2.2, R28.1
- removed net N$19: 4017A.Q4, 4017A.RES
- removed net N$20: DIS1.CONTR, POT4.WIPER
- removed net N$21: D3.A, IC1.1Y
- removed net N$22: D4.A, IC1.2Y
- removed net N$23: D4.C, D5.A, X2-2.KL
- removed net N$24: D2.A, D3.C, X2-1.KL
- removed net N$25: D6.A, X3-1.KL
- removed net N$27: DZ1-3.C, R11.1
- removed net N$28: DZ1-5.C, R13.1
- removed net N$29: DZ1-1.C, R8.1
- removed net N$30: DZ1-2.C, R10.1
- removed net N$31: DZ1-4.C, R12.1
- removed net N$32: DZ1-6.C, R14.1
- removed net N$33: DZ1-7.C, R15.1
- removed net N$34: DZ1-8.C, R16.1
- removed net N$35: DZ1-9.C, R17.1
- removed net N$36: DZ1-10.C, R18.1
- removed net N$37: LED1.A, R22.2
- removed net N$38: R21.1, R9.2, U$2.SQW
- removed net N$39: Q2.B, R5.1
- removed net N$40: R21.2, T3.B
- removed net N$41: LED1.C, T3.C
- removed net N$42: D1.C, K11.2
- removed net RST: PINGUINO.RST, RESET.S, RESET.S1
- new net 12V: C5.1, IC1.VI, R1.1
- new net 12V1: C7.1, C8.+, IC1.VO, IC2.VI, L2.2
- new net 3V3: C12.1, L4.1, LED3.A
- new net 5V: C9.1, L3.1, LED2.A
- new net 6V: C6.1, L2.1, LED1.A
- new net N$26: PINGUINOBASE.PIN12-PWM
- new net N$43: PINGUINOBASE.PIN11-PWM
- new net N$44: PINGUINOBASE.PIN10
- new net N$45: PINGUINOBASE.RST
- new net N$46: PINGUINOBASE.GND
- new net N$47: PINGUINOBASE.+5V
- new net N$48: PINGUINOBASE.PIN20/ANALOG-7
- new net N$49: PINGUINOBASE.PIN19/ANALOG-6
- new net N$50: PINGUINOBASE.PIN18/ANALOG-5
- new net N$51: PINGUINOBASE.PIN17/ANALOG-4
- new net N$52: PINGUINOBASE.PIN16/ANALOG-3
- new net N$53: PINGUINOBASE.PIN15/ANALOG-2
- new net N$54: PINGUINOBASE.PIN14/ANALOG-1
- new net N$55: PINGUINOBASE.PIN13/ANALOG-0
- new net N$57: C1.1, C2.+, F1.2, L1.1
- new net N$6: PINGUINOBASE.PIN22
- net GND: now also C10.2, C11.-, C12.2, C13.2, C14.-, C3.2, C4.-, C5.2, C6.2, C7.2, C8.-, C9.2, IC1.GND, IC3.GND, J1.2, J1.3, R2.1, R4.1; no longer 4017A.ENA, 4017P.VSS, BAT1.-, C3.-, C4.2, DIS1.D0, DIS1.D1, DIS1.D2, DIS1.D3, DIS1.GND, DIS1.NC@2, DIS1.R/W, IC1.3-4EN, IC1.3A, IC1.4A, IC1.GND1, IC1.GND2, IC1.GND3, IC1.GND4, IC2.A0, IC2.A1, IC2.A2, IC2.WP, IC5.GND, JP1.2, LM35.GND, PINGUINO.GND, POT1.CW, POT2.CW, POT3.CW, POT4.CW, Q2.C, R10.2, R11.2, R12.2, R13.2, R14.2, R15.2, R16.2, R17.2, R18.2, R20.1, R8.2, RESET.P, RESET.P1, T2.E, T3.E, U$2.GND, X3-2.KL
- net N$1: now also F1.1, J1.1; no longer LM35.VO, R1.1
- net N$2: now also C3.1, C4.+, L1.2, R1.2; no longer Q1.2, U$2.X1
- net N$3: now also C10.1, C11.+, IC2.VO, IC3.VI, L3.2; no longer Q1.1, U$2.X2
- net N$4: now also C13.1, C14.+, IC3.VO, L4.2; no longer 4017A.Q0, U$1.C4
- net N$5: now also LED2.C, R3.2; no longer BAT1.+, U$2.VBATT
- net N$7: now also PINGUINOBASE.PIN21; no longer IC3.ADJ, R3.2, R4.2
- net N$8: now also LED1.C, R2.2; no longer 4017A.Q1, U$1.C3
- net N$9: now also LED3.C, R4.2; no longer K12.P, X1-2.KL
Other:
- note removed: "AN Libre"
- note removed: "ENTRENADORA PARA"
- note removed: "Fotoresistencia"
- note removed: "GND"
- note removed: "LED9/BUZZER"
- note removed: "LM35"
- note removed: "MOTOR"
- note removed: "MOTOR-PWM"
- note removed: "PINGUINO BASE"
- note removed: "POT1"
- note removed: "POT2"
- note removed: "POT3"
- note removed: "Photocelda"
- note removed: "RESET"
- note removed: "Sensor Temperatura (LM35)"
- note removed: "Teclado R1"
- note removed: "Teclado R2"
- note removed: "Teclado R3"
- note removed: "Teclado R4"
- note removed: "V+"
- moved on the sheet: C1, C2, LED1, R1, R2, R3, R4

Commit message: Algunas actualizaciones al cableado de la lcd 16x2
Parts:
- removed C10, C12, C13, C5, C6, C7, C9: 100nf, rcl:C-EU050-024X044
- removed C11, C14, C8: 100uf, rcl:CPOL-USE2.5-5
- removed F1: 2amp, special:FUSE
- removed J1: (no value), con-jack:DCJ0303
- removed L1, L2, L3, L4: 100uH, rcl:L-EU0207/10
- removed LED2, LED3: (no value), adafruit:LED3MM
- added BAT1: (no value), SparkFun:BATTERY20PTH
- added D1: 1N4007, adafruit:1N4004
- added D2, D3, D4, D5: 1N4007, diode:1N4148DO35-7
- added D6: 4007, diode:1N4148DO35-7
- added DZ1: LB10, led:LB10
- added I2C, UART: (no value), SparkFun:M04LONGPADS
- added IC4: 74LS155N, 74xx-us:74LS155N
- added IC5: 7805, v-reg:78XXL
- added JP1: Sensores Externos, SparkFun:M06LONGPADS
- added JP2: (no value), SparkFun:M02PTH3
- added K1: CQ1-12V, relay:CQ1-12V
- added LM35: LM35CZ, lm35:LM35CZ
- added POT1, POT2, POT3, POT5: 5k, SparkFun:TRIMPOTPTH
- added Q1: (no value), crystal:CRYSTALTC38H
- added Q2: 2N2222, SparkFun:TRANSISTOR_NPNTO92
- added R10, R11, R12, R13, R14, R15, R16, R17, R18, R8: 470, SparkFun:RESISTORKIT
- added R19: PHOTOCELLPTH, SparkFun:PHOTOCELLPTH
- added R20: 10k, rcl:R-US_0204/5
- added R21, R22, R24, R28, R7, R9: 4.7k, SparkFun:RESISTORKIT
- added R29: 1k, SparkFun:RESISTORKIT
- added R5, R6: 1k, rcl:R-EU_0204/7
- added RESET: (no value), switch-omron:10-XX
- added SERVOS, SERVOS1: (no value), SparkFun:M03LONGPADS
- added SG1: BUZZERPTH, SparkFun:BUZZERPTH
- added T1, T2: 2N3904, transistor:2N3904
- added T3: 2SC1815, transistor:2SC1815
- added U$1: (no value), keypad4x4_ece:KEYPAD4X4
- added U$2: XBEE, adafruit:XBEE
- added U$4: DS1307, aasanchez:DS1307
- added U1: LCD-16X2SILK, SparkFun:LCD-16X2SILK
- added X1: (no value), con-wago-508:W237-3E
- added X2, X3: (no value), con-wago-508:W237-02P
- added XB1: XBEE-PRO, maxstream:XBEE-PRO
- C1: value 100nf -> 0.1uf; device rcl:C-EU050-024X044 -> SparkFun:CAPPTH2
- C2: value 470uf -> 220nf; device rcl:CPOL-USE2.5-7 -> SparkFun:CAP_POLPTH2
- C3: value 100nf -> 0.33uf/50v; device rcl:C-EU050-024X044 -> SparkFun:CAP_POLPTH2
- C4: value 100uf -> 0.1uf; device rcl:CPOL-USE2.5-5 -> SparkFun:CAPPTH2
- IC1: value 7806T -> L293B; device adafruit:7806T -> st-microelectronics:L293D
- IC2: value 7805T -> 24AA64P; device adafruit:7806T -> microchip:24AA64P
- IC3: value 7803T -> lm317; device adafruit:7806T -> v-reg:LM317TL
- PINGUINOBASE: value PINGUINOBASENO-BORDER -> PINGUINOBASEFACEDOWN; device PinguinoBase:PINGUINOBASENO-BORDER -> PinguinoBase:PINGUINOBASEFACEDOWN
- R1: value 4.7Ohm/2w -> 1k; device rcl:R-US_0414/15 -> SparkFun:RESISTORKIT
- R2: value (none) -> 4.7k
- R3: value (none) -> 360
- R4: value (none) -> 240
Connections:
- removed net 12V: C5.1, IC1.VI, R1.1
- removed net 12V1: C7.1, C8.+, IC1.VO, IC2.VI, L2.2
- removed net 3V3: C12.1, L4.1, LED3.A
- removed net 6V: C6.1, L2.1, LED1.A
- removed net N$26: PINGUINOBASE.PIN12-PWM
- removed net N$4: C13.1, C14.+, IC3.VO, L4.2
- removed net N$43: PINGUINOBASE.PIN11-PWM
- removed net N$44: PINGUINOBASE.PIN10
- removed net N$49: PINGUINOBASE.PIN19/ANALOG-6
- removed net N$50: PINGUINOBASE.PIN18/ANALOG-5
- removed net N$51: PINGUINOBASE.PIN17/ANALOG-4
- removed net N$52: PINGUINOBASE.PIN16/ANALOG-3
- removed net N$53: PINGUINOBASE.PIN15/ANALOG-2
- removed net N$54: PINGUINOBASE.PIN14/ANALOG-1
- removed net N$55: PINGUINOBASE.PIN13/ANALOG-0
- removed net N$57: C1.1, C2.+, F1.2, L1.1
- removed net N$8: LED1.C, R2.2
- new net !10: IC1.2A, Q2.E, R6.1
- new net +12V: C2.+, C3.+, D2.C, D5.C, D6.C, IC1.VCC2, IC5.IN
- new net +3V3: IC3.OUT, JP1.1, R4.1, XB1.VCC
- new net +5V: C1.1, C4.1, IC1.VCC1, IC2.VCC, IC3.IN, IC5.OUT, JP1.3, LM35.+VS, POT1.CCW, POT2.CCW, POT3.CCW, R19.P$2, R2.2, R22.1, R29.2, R6.2, R7.2, R9.1, SG1.1, U$4.VCC
- new net 0: IC2.SCL, PINGUINOBASE.SDA-PIN0, R2.1, U$4.SCL
- new net 1: IC2.SDA, PINGUINOBASE.SCL-PIN1, R7.1, U$4.SDA
- new net 10: IC1.1A, R5.2
- new net 11: DZ1-1.A, IC1.1-2EN
- new net 12: DZ1-2.A, JP2.1
- new net 13: R19.P$1, R20.2
- new net 14: R1.2
- new net 15: JP1.6
- new net 16: JP1.5
- new net 17: JP1.4
- new net 18: POT1.WIPER
- new net 19: POT2.WIPER
- new net 2: IC4A.B, PINGUINOBASE.PIN2, R24.1
- new net 20: POT3.WIPER
- new net 21: DZ1-3.A
- new net 22: DZ1-4.A, PINGUINOBASE.PIN22, U1.RS
- new net 23: DZ1-5.A, PINGUINOBASE.PIN23, U1.A
- new net 24: DZ1-6.A, PINGUINOBASE.PIN24, U1.DB7
- new net 25: DZ1-7.A, PINGUINOBASE.PIN25, U1.DB6
- new net 26: DZ1-8.A, PINGUINOBASE.PIN26, U1.DB5
- new net 27: DZ1-9.A, PINGUINOBASE.PIN27, U1.DB4
- new net 28: DZ1-10.A, PINGUINOBASE.PIN28, U1.E
- new net 3: IC4A.A, PINGUINOBASE.PIN3
- new net 4: PINGUINOBASE.PIN4, U$1.C1
- new net 5: PINGUINOBASE.PIN5, U$1.C2
- new net 6: PINGUINOBASE.PIN6, U$1.C3
- new net 7: PINGUINOBASE.PIN7, U$1.C4
- new net 8: UART.1
- new net 9: UART.2
- new net N$10: K12.O, X1-3.KL
- new net N$11: K12.S, X1-1.KL
- new net N$12: R24.2, T1.B
- new net N$14: R28.2, T2.B
- new net N$15: D1.A, K11.1, T1.C
- new net N$16: R29.1, SG1.2, T2.C
- new net N$18: JP2.2, R28.1
- new net N$21: D3.A, IC1.1Y
- new net N$22: D4.A, IC1.2Y
- new net N$23: D4.C, D5.A, X2-2.KL
- new net N$24: D2.A, D3.C, X2-1.KL
- new net N$25: D6.A, X3-1.KL
- new net N$27: DZ1-3.C, R11.1
- new net N$28: DZ1-5.C, R13.1
- new net N$29: DZ1-1.C, R8.1
- new net N$30: DZ1-2.C, R10.1
- new net N$31: DZ1-4.C, R12.1
- new net N$32: DZ1-6.C, R14.1
- new net N$33: DZ1-7.C, R15.1
- new net N$34: DZ1-8.C, R16.1
- new net N$35: DZ1-9.C, R17.1
- new net N$36: DZ1-10.C, R18.1
- new net N$37: LED1.A, R22.2
- new net N$38: R21.1, R9.2, U$4.SQW
- new net N$39: Q2.B, R5.1
- new net N$40: R21.2, T3.B
- new net N$41: LED1.C, T3.C
- new net N$42: D1.C, K11.2
- new net RST: RESET.S, RESET.S1
- net 5V: now also PINGUINOBASE.+5V, POT5.CCW, U1.VDD; no longer C9.1, L3.1, LED2.A
- net GND: now also BAT1.-, C3.-, C4.2, IC1.3-4EN, IC1.3A, IC1.4A, IC1.GND1, IC1.GND2, IC1.GND3, IC1.GND4, IC2.A0, IC2.A1, IC2.A2, IC2.WP, IC5.GND, JP1.2, LM35.GND, PINGUINOBASE.GND, POT1.CW, POT2.CW, POT3.CW, POT5.CW, Q2.C, R10.2, R11.2, R12.2, R13.2, R14.2, R15.2, R16.2, R17.2, R18.2, R20.1, R8.2, RESET.P, RESET.P1, T2.E, T3.E, U$4.GND, U1.DB0, U1.DB1, U1.DB2, U1.DB3, U1.K, U1.R/W, U1.VSS, X3-2.KL; no longer C10.2, C11.-, C12.2, C13.2, C14.-, C3.2, C4.-, C5.2, C6.2, C7.2, C8.-, C9.2, IC1.GND, IC3.GND, J1.2, J1.3, R2.1, R4.1
- net N$1: now also LM35.VO, R1.1; no longer F1.1, J1.1
- net N$2: now also Q1.2, U$4.X1; no longer C3.1, C4.+, L1.2, R1.2
- net N$3: now also Q1.1, U$4.X2; no longer C10.1, C11.+, IC2.VO, IC3.VI, L3.2
- net N$45: now also IC4A.1Y3, U$1.R4; no longer PINGUINOBASE.RST
- net N$46: now also IC4A.1Y2, U$1.R3; no longer PINGUINOBASE.GND
- net N$47: now also IC4A.1Y1, U$1.R2; no longer PINGUINOBASE.+5V
- net N$48: now also IC4A.1Y0, U$1.R1; no longer PINGUINOBASE.PIN20/ANALOG-7
- net N$5: now also BAT1.+, U$4.VBATT; no longer LED2.C, R3.2
- net N$6: now also POT5.WIPER, U1.VO; no longer PINGUINOBASE.PIN22
- net N$7: now also IC3.ADJ, R3.2, R4.2; no longer PINGUINOBASE.PIN21
- net N$9: now also K12.P, X1-2.KL; no longer LED3.C, R4.2
Other:
- note added: "ENTRENADORA PARA"
- note added: "Fotoresistencia"
- note added: "PINGUINO BASE"
- note added: "Sensor Temperatura (LM35)"
- moved on the sheet: C1, C2, LED1, R1, R2, R3, R4
